File: Switches.kicad_sch (KiCad schematic)
At the start: 30 parts, among them SW1 PEC11R, SW2 SW_SPST, SW3 SW_SPST, SW4 PEC11R, SW5 SW_SPST, SW6 SW_SPST, SW7 PEC11R, SW8 SW_SPST, SW9 SW_SPST

Commit message: remove crumbcatcher name from files
Other:
- title: Crumb Catcher -> Mad 2040
Changed lines of the file:
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@@
 	(paper "A4")
 	(title_block
-		(title "Crumb Catcher")
+		(title "Mad 2040")
 		(date "2023-10-25")
 		(rev "A")
