File: MCU_RP2040.kicad_sch (KiCad schematic)
At the start: 35 parts, among them Q1 2N7002PV,115, X1 ECS-2520MVLC-120-CN

Commit message: BOM update
Parts:
- C19, C20, C21, C7, C? (x8): LCSC PN (none) -> C432917
- C8, C?: LCSC PN (none) -> C472857
- SW?: LCSC PN (none) -> C79147
- X1: LCSC PN (none) -> C17361989
Changed lines of the file:
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@@
 			)
 		)
+		(property "LCSC PN" "C432917"
+			(at 142.24 35.56 0)
+			(effects
+				(font
+					(size 1.27 1.27)
+				)
+				(hide yes)
+			)
+		)
 		(pin "1"
 		)
@@
 			)
 		)
+		(property "LCSC PN" "C472857"
+			(at 93.98 181.61 0)
+			(effects
+				(font
+					(size 1.27 1.27)
+				)
+				(hide yes)
+			)
+		)
 		(pin "2"
 		)
@@
 			)
 		)
+		(property "LCSC PN" "C432917"
+			(at 107.95 35.56 0)
+			(effects
+				(font
+					(size 1.27 1.27)
+				)
+				(hide yes)
+			)
+		)
 		(pin "1"
 		)
@@
 			)
 		)
+		(property "LCSC PN" "C17361989"
+			(at 72.39 74.93 0)
+			(effects
+				(font
+					(size 1.27 1.27)
+				)
+				(hide yes)
+			)
+		)
 		(pin "3"
 		)
@@
 			)
 		)
+		(property "LCSC PN" "C432917"
+			(at 119.38 35.56 0)
+			(effects
+				(font
+					(size 1.27 1.27)
+				)
+				(hide yes)
+			)
+		)
 		(pin "1"
 		)
@@
 			)
 		)
+		(property "LCSC PN" "C432917"
+			(at 54.61 115.57 0)
+			(effects
+				(font
+					(size 1.27 1.27)
+				)
+				(hide yes)
+			)
+		)
 		(pin "1"
 		)
@@
 			)
 		)
+		(property "LCSC PN" "C432917"
+			(at 153.67 35.56 0)
+			(effects
+				(font
+					(size 1.27 1.27)
+				)
+				(hide yes)
+			)
+		)
 		(pin "1"
 		)
@@
 			)
 		)
+		(property "LCSC PN" "C432917"
+			(at 224.79 35.56 0)
+			(effects
+				(font
+					(size 1.27 1.27)
+				)
+				(hide yes)
+			)
+		)
 		(pin "1"
 		)
@@
 			)
 		)
+		(property "LCSC PN" "C432917"
+			(at 55.88 76.2 0)
+			(effects
+				(font
+					(size 1.27 1.27)
+				)
+				(hide yes)
+			)
+		)
 		(pin "1"
 		)
@@
 			)
 		)
+		(property "LCSC PN" "C432917"
+			(at 165.1 35.56 0)
+			(effects
+				(font
+					(size 1.27 1.27)
+				)
+				(hide yes)
+			)
+		)
 		(pin "1"
 		)
@@
 			)
 		)
+		(property "LCSC PN" "C432917"
+			(at 130.81 35.56 0)
+			(effects
+				(font
+					(size 1.27 1.27)
+				)
+				(hide yes)
+			)
+		)
 		(pin "1"
 		)
@@
 			)
 		)
+		(property "LCSC PN" "C432917"
+			(at 215.9 35.56 0)
+			(effects
+				(font
+					(size 1.27 1.27)
+				)
+				(hide yes)
+			)
+		)
 		(pin "1"
 		)
@@
 			)
 		)
+		(property "LCSC PN" "C432917"
+			(at 187.96 35.56 0)
+			(effects
+				(font
+					(size 1.27 1.27)
+				)
+				(hide yes)
+			)
+		)
 		(pin "1"
 		)
@@
 			)
 		)
+		(property "LCSC PN" "C79147"
+			(at 40.64 172.72 0)
+			(effects
+				(font
+					(size 1.27 1.27)
+				)
+				(hide yes)
+			)
+		)
 		(pin "1"
 		)
@@
 			)
 		)
+		(property "LCSC PN" "C432917"
+			(at 176.53 35.56 0)
+			(effects
+				(font
+					(size 1.27 1.27)
+				)
+				(hide yes)
+			)
+		)
 		(pin "1"
 		)
@@
 			(at 83.82 181.61 0)
 			(effects
+				(font
+					(size 1.27 1.27)
+				)
+				(hide yes)
+			)
+		)
+		(property "LCSC PN" "C472857"
+			(at 83.82 181.61 0)
+			(effects

Commit message: BOM consolidation
Parts:
- removed R?: 100K, Resistor_SMD:R_0402_1005Metric, symbol Device:R_Small
- removed R? (x2): 27R, Resistor_SMD:R_0402_1005Metric, symbol Device:R_Small
- added R15, R9: 51K, Resistor_SMD:R_0402_1005Metric, symbol Device:R_Small
- C8, C?: LCSC PN C472857 -> C2932476
- U?: footprint Package_SO:SOIC-8_5.23x5.23mm_P1.27mm -> Mad_Footprints:SOIC-8_5.23x5.23mm_P1.27mm
Connections:
- net GND: now also R15.2
- net USB_D+: now also U?.47 (D+)
- net USB_D-: now also U?.46 (D-)
- net at C8.1, C?.1, Q?.5 (G)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: now also R9.1
- new net: R15.1, R9.2

Commit message: BOM update
Parts:
- C19, C20, C21, C7, C? (x8): LCSC (none) -> C432917; LCSC PN C432917 -> (none)
- C8, C?: LCSC (none) -> C2932476; LCSC PN C2932476 -> (none)
- C? (x2): LCSC (none) -> C14664; LCSC PN C14664 -> (none)
- D?: symbol PCM_Diode_Schottky_AKL:RB520S30 -> Mad_Symbols:RB520S30; LCSC (none) -> C232575; LCSC PN C232575 -> (none)
- Q1, Q?: LCSC (none) -> C551422; LCSC PN C551422 -> (none)
- R10, R?: LCSC (none) -> C106235; LCSC PN C106235 -> (none)
- R15, R9, R?: LCSC (none) -> C107229; LCSC PN C107229 -> (none)
- R? (x3): LCSC (none) -> C60490; LCSC PN C60490 -> (none)
- SW?: LCSC (none) -> C79147; LCSC PN C79147 -> (none)
- U?: LCSC (none) -> C2040; LCSC PN C2040 -> (none)
- U?: LCSC (none) -> C97521; LCSC PN C97521 -> (none)
- X1: footprint Mad_Footprints:Crystal_SMD_ECX-32-4Pin_3.2x2.5mm -> Mad_Footprints:Oscillator_SMD_ECS_2520MV-xxx-xx-4Pin_2.5x2.0mm; LCSC (none) -> C669073; LCSC PN C17361989 -> (none)
Other:
- note removed: "Check Pinout"
- moved on the sheet: C20, C8, C?, Q?B, R15, R9, R?, TP?
