File: Mad_RP2040.kicad_pcb (KiCad board)
At the start: 2 copper layers, 38 x 32.1 mm, 64 parts, among them J1 USB_C_Receptacle, J2 Conn_ARM_SWD_TagConnect_TC203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, Q1 2N7002PV,115, SW1 SW_SPST, SW2 SW_SPST, SW3 EVPAA202K, U0 PCB, U1 ECMF02-2AMX6, U3 NCP1117-3.3, U4 W25Q128JVSIQ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

Commit message: BOM update
Parts:
- X1: footprint Mad_Footprints:Crystal_SMD_ECX-32-4Pin_3.2x2.5mm -> Mad_Footprints:Oscillator_SMD_ECS_2520MV-xxx-xx-4Pin_2.5x2.0mm

Commit message: Update design rules
Parts:
- moved Q1 0.45 mm to (158.2, 82.7)
- moved R12 0.45 mm to (157.4, 85.2)
- moved R6 0.45 mm to (158.8, 84.7)
- moved R7 0.45 mm to (158.1, 80.7)
- moved SW3 0.45 mm to (158.3, 88.5)
- moved X1 0.25 mm to (158.0, 78.5), turned to 180 degrees
Routing:
- net VBUS: track 0.00 -> 10.9 mm
- net /PreFIlterGND: track 0.00 -> 3.88 mm
- net /RP2040/3V3: track 16.7 -> 13.2 mm
- net Net-(X1-OUT): track 1.33 -> 0.00 mm
Changed lines of the file:
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@@
 	(footprint "Mad_Footprints:Oscillator_SMD_ECS_2520MV-xxx-xx-4Pin_2.5x2.0mm"
 		(layer "B.Cu")
-		(at 158.15 78.375 -90)
+		(at 157.975 78.55 180)
 		(descr "Miniature Crystal Clock Oscillator ECS 2520MV series, https://www.ecsxtal.com/store/pdf/ECS-2520MV.pdf")
 		(tags "Miniature Crystal Clock Oscillator ECS 2520MV series SMD SMT HCMOS")
 		(property "Reference" "X1"
-			(at 0 2.5 -90)
+			(at 0 2.5 180)
 			(layer "B.SilkS")
 			(effects
@@
 		)
 		(property "Value" "ECS-2520MVLC-120-CN"
-			(at 0 -2.5 -90)
+			(at 0 -2.5 180)
 			(layer "B.Fab")
 			(effects
@@
 		)
 		(property "Footprint" "Mad_Footprints:Oscillator_SMD_ECS_2520MV-xxx-xx-4Pin_2.5x2.0mm"
-			(at 0 0 90)
+			(at 0 0 0)
 			(unlocked yes)
 			(layer "B.Fab")
@@
 		)
 		(property "Datasheet" "https://www.ecsxtal.com/store/pdf/ECS-2520MV.pdf"
-			(at 0 0 90)
+			(at 0 0 0)
 			(unlocked yes)
 			(layer "B.Fab")
@@
 		)
 		(property "Description" "12 MHz XO (Standard) CMOS Oscillator 1.6V ~ 3.6V Enable/Disable 4-SMD, No Lead"
-			(at 0 0 90)
+			(at 0 0 0)
 			(unlocked yes)
 			(layer "B.Fab")
@@
 		)
 		(property "Price" "$1.99"
-			(at 0 0 90)
+			(at 0 0 0)
 			(unlocked yes)
 			(layer "B.Fab")
@@
 		)
 		(property "Interface" ""
-			(at 0 0 90)
+			(at 0 0 0)
 			(unlocked yes)
 			(layer "B.Fab")
@@
 		)
 		(property "Rating" "XTAL OSC XO 12.0000MHZ CMOS SMD"
-			(at 0 0 90)
+			(at 0 0 0)
 			(unlocked yes)
 			(layer "B.Fab")
@@
 		)
 		(property "Supplier" "Digikey"
-			(at 0 0 90)
+			(at 0 0 0)
 			(unlocked yes)
 			(layer "B.Fab")
@@
 		)
 		(property "Supplier PN" "50-ECS-2520MVLC-120-CN-TRCT-ND"
-			(at 0 0 90)
+			(at 0 0 0)
 			(unlocked yes)
 			(layer "B.Fab")
@@
 		)
 		(property "Manufacturer" "ECS Inc."
-			(at 0 0 90)
+			(at 0 0 0)
 			(unlocked yes)
 			(layer "B.Fab")
@@
 		)
 		(property "MPN" "ECS-2520MVLC-120-CN-TR"
-			(at 0 0 90)
+			(at 0 0 0)
 			(unlocked yes)
 			(layer "B.Fab")
@@
 		)
 		(property "Substitute" ""
-			(at 0 0 -90)
+			(at 0 0 180)
 			(unlocked yes)
 			(layer "B.Fab")
@@
 		)
 		(property "LCSC" "C669073"
-			(at 0 0 -90)
+			(at 0 0 180)
 			(unlocked yes)
 			(layer "B.Fab")
@@
 		(attr smd)
 		(fp_line
-			(start -1.07 1.56)
-			(end -0.38 1.56)
+			(start 1.11 0.32)
+			(end 1.11 -0.32)
 			(stroke
 				(width 0.12)
@@
 		)
 		(fp_line
-			(start -1.11 0.32)
-			(end -1.11 -0.32)
+			(start 0.17 -1.36)
+			(end -0.17 -1.36)
 			(stroke
 				(width 0.12)
@@
 		)
 		(fp_line
-			(start 1.11 0.32)
-			(end 1.11 -0.32)
+			(start -1.07 1.56)
+			(end -0.38 1.56)
 			(stroke
 				(width 0.12)
@@
 		)
 		(fp_line
-			(start 0.17 -1.36)
-			(end -0.17 -1.36)
+			(start -1.11 0.32)
+			(end -1.11 -0.32)
 			(stroke
 				(width 0.12)
@@
 		)
 		(fp_line
-			(start -1.38 -1.63)
-			(end -1.38 1.63)
+			(start 1.38 -1.63)
+			(end 1.38 1.63)
 			(stroke
 				(width 0.05)
@@
 		(fp_line
 			(start 1.38 -1.63)
-			(end 1.38 1.63)
+			(end -1.38 -1.63)
 			(stroke
 				(width 0.05)
@@
 		)
 		(fp_line
-			(start 1.38 -1.63)
-			(end -1.38 -1.63)
+			(start -1.38 -1.63)
+			(end -1.38 1.63)
 			(stroke
 				(width 0.05)
@@
 		)
 		(fp_line
-			(start -0.5 1.25)
-			(end -1 0.75)
+			(start 1 1.25)
+			(end -0.5 1.25)
 			(stroke
 				(width 0.1)
@@
 		)
 		(fp_line
-			(start 1 1.25)
-			(end -0.5 1.25)
+			(start 1 -1.25)
+			(end 1 1.25)
 			(stroke
 				(width 0.1)
@@
 		)
 		(fp_line
-			(start -1 -1.25)
-			(end -1 0.75)
+			(start 1 -1.25)
+			(end -1 -1.25)
 			(stroke
 				(width 0.1)
@@
 		)
 		(fp_line
-			(start 1 -1.25)
-			(end 1 1.25)
+			(start -0.5 1.25)
+			(end -1 0.75)
 			(stroke
 				(width 0.1)
@@
 		)
 		(fp_line
-			(start 1 -1.25)
-			(end -1 -1.25)
+			(start -1 -1.25)
+			(end -1 0.75)
 			(stroke
 				(width 0.1)
@@
 		)
 		(fp_text user "${REFERENCE}"
-			(at 0 0 0)
+			(at 0 0 270)
 			(layer "B.Fab")
 			(effects
@@
 		)
 		(pad "1" smd roundrect
-			(at -0.725 0.925 270)
+			(at -0.725 0.925 180)
 			(size 0.8 0.9)
 			(layers "B.Cu" "B.Paste" "B.Mask")
@@
 		)
 		(pad "2" smd roundrect
-			(at -0.725 -0.925 270)
+			(at -0.725 -0.925 180)
 			(size 0.8 0.9)
 			(layers "B.Cu" "B.Paste" "B.Mask")
@@
 		)
 		(pad "3" smd roundrect
-			(at 0.725 -0.925 270)
+			(at 0.725 -0.925 180)
 			(size 0.8 0.9)
 			(layers "B.Cu" "B.Paste" "B.Mask")
@@
 		)
 		(pad "4" smd roundrect
-			(at 0.725 0.925 270)
+			(at 0.725 0.925 180)
 			(size 0.8 0.9)
 			(layers "B.Cu" "B.Paste" "B.Mask")
@@
 	(footprint "Resistor_SMD:R_0402_1005Metric"
 		(layer "B.Cu")
-		(at 158.05 81.175 180)
+		(at 158.05 80.725 180)
 		(descr "Resistor SMD 0402 (1005 Metric), square (rectangular) end terminal, IPC_7351 nominal, (Body size source: IPC-SM-782 page 72, https://www.pcb-3d.com/wordpress/wp-content/uploads/ipc-sm-782a_amendment_1_and_2.pdf), generated with kicad-footprint-generator")
 		(tags "resistor")
@@
 	(footprint "Package_TO_SOT_SMD:SOT-666"
 		(layer "B.Cu")
-		(at 158.15 83.175 90)
+		(at 158.15 82.725 90)
 		(descr "SOT666")
 		(tags "SOT-666")
@@
 	(footprint "Mad_Footprints:EVP-AA202K"
 		(layer "B.Cu")
-		(at 158.35 88.975 90)
+		(at 158.35 88.525 90)
 		(descr "Tactile Switch SPST-NO Top Actuated Surface Mount")
 		(tags "SWITCH TACTILE SPST-NO")
@@
 	(footprint "Resistor_SMD:R_0402_1005Metric"
 		(layer "B.Cu")
-		(at 158.85 85.175 180)
+		(at 158.85 84.725 180)
 		(descr "Resistor SMD 0402 (1005 Metric), square (rectangular) end terminal, IPC_7351 nominal, (Body size source: IPC-SM-782 page 72, https://www.pcb-3d.com/wordpress/wp-content/uploads/ipc-sm-782a_amendment_1_and_2.pdf), generated with kicad-footprint-generator")
 		(tags "resistor")
@@
 	(footprint "Resistor_SMD:R_0402_1005Metric"
 		(layer "B.Cu")
-		(at 157.45 85.675 -90)
+		(at 157.45 85.225 -90)
 		(descr "Resistor SMD 0402 (1005 Metric), square (rectangular) end terminal, IPC_7351 nominal, (Body size source: IPC-SM-782 page 72, https://www.pcb-3d.com/wordpress/wp-content/uploads/ipc-sm-782a_amendment_1_and_2.pdf), generated with kicad-footprint-generator")
 		(tags "resistor")
@@
 	)
 	(segment
-		(start 158.845 77.02)
-		(end 159.05 77.225)
-		(width 0.25)
-		(layer "B.Cu")
-		(net 2)
-	)
-	(segment
 		(start 145.23 81.075)
 		(end 145.25 81.075)
@@
 	)
 	(segment
-		(start 156.025 77.02)
-		(end 158.845 77.02)
-		(width 0.25)
-		(layer "B.Cu")
-		(net 2)
-	)
-	(segment
 		(start 151.55 83.0125)
 		(end 151.55 84.095)
@@
 	)
 	(segment
-		(start 155.75 77.295)
-		(end 156.025 77.02)
-		(width 0.25)
-		(layer "B.Cu")
-		(net 2)
-	)
-	(segment
 		(start 144.525 82.175)
 		(end 144.9989 81.7011)
@@
 	)
 	(segment
+		(start 129.65 81.49)
+		(end 129.95 81.79)
+		(width 0.25)
+		(layer "B.Cu")
+		(net 11)
+	)
+	(segment
+		(start 128.890364 77.8526)
+		(end 129.65 78.612236)
+		(width 0.25)
+		(layer "B.Cu")
+		(net 11)
+	)
+	(segment
+		(start 124.85 79.105)
+		(end 124.85 78.529949)
+		(width 0.25)
+		(layer "B.Cu")
+		(net 11)
+	)
+	(segment
+		(start 129.65 79.105)
+		(end 129.65 81.49)
+		(width 0.25)
+		(layer "B.Cu")
+		(net 11)
+	)
+	(segment
+		(start 124.93 79.185)
+		(end 124.85 79.105)
+		(width 0.25)
+		(layer "B.Cu")
+		(net 11)
+	)
+	(segment
+		(start 124.93 80.665)
+		(end 124.93 79.185)
+		(width 0.25)
+		(layer "B.Cu")
+		(net 11)
+	)
+	(segment
+		(start 125.527349 77.8526)
+		(end 128.890364 77.8526)
+		(width 0.25)
+		(layer "B.Cu")
+		(net 11)
+	)
+	(segment
+		(start 124.85 78.529949)
+		(end 125.527349 77.8526)
+		(width 0.25)
+		(layer "B.Cu")
+		(net 11)
+	)
+	(segment
+		(start 129.65 78.612236)
+		(end 129.65 79.105)
+		(width 0.25)
+		(layer "B.Cu")
+		(net 11)
+	)
+	(segment
 		(start 127.425 81.425)
 		(end 127.425 79.9689)
@@
 	)
 	(segment
-		(start 156.9 79.175)
-		(end 157.25 79.525)
+		(start 127.925 81.77474)
+		(end 127.62474 82.075)
+		(width 0.25)
+		(layer "B.Cu")
+		(net 25)
+	)
+	(segment
+		(start 127.925 81.425)
+		(end 127.925 81.77474)
 		(width 0.25)
 		(layer "B.Cu")
-		(net 24)
+		(net 25)
+	)
+	(segment
+		(start 127.62474 82.075)
+		(end 126.275 82.075)
+		(width 0.25)
+		(layer "B.Cu")
+		(net 25)
+	)
+	(segment
+		(start 127.925 81.425)
+		(end 128.8 81.425)
+		(width 0.25)
+		(layer "B.Cu")
+		(net 25)
 	)
 	(segment
-		(start 156.06 79.175)
-		(end 156.9 79.175)
+		(start 126.275 82.075)
+		(end 125.85 81.65)
 		(width 0.25)
 		(layer "B.Cu")
-		(net 24)
+		(net 25)
+	)
+	(segment
+		(start 128.8 81.425)
+		(end 129 81.625)
+		(width 0.25)
+		(layer "B.Cu")
+		(net 25)
 	)
 	(segment
@@
 		(priority 2)
 		(connect_pads yes
-			(clearance 0.5)
+			(clearance 0.3)
 		)
 		(min_thickness 0.25)

Commit message: Add dru, start routing
Parts:
- moved R11 1.87 mm to (157.9, 86.6), turned to 0 degrees
- moved SW3 1.23 mm to (158.1, 89.7), turned to -90 degrees
- moved C20 0.60 mm to (155.2, 80.9)
- moved C10 0.35 mm to (147.8, 74.5)
- moved C7 0.35 mm to (156.1, 77.8)
- moved C17 0.30 mm to (151.8, 74.5)
- moved C18 0.20 mm to (156.1, 80.6)
- moved C8 0.08 mm to (154.1, 86.7)
- turned D1 to 0 degrees
- turned D2 to 0 degrees
Routing:
- net GND: track 11.1 -> 51.5 mm, vias 0 -> 40
- net /RP2040/3V3: track 13.2 -> 41.2 mm, vias 0 -> 12
- net +5V: track 0.00 -> 19.0 mm, vias 0 -> 3
- net Net-(Q1B-G): track 0.00 -> 10.5 mm
- net Net-(D7-A): track 0.00 -> 10.5 mm
- net Net-(D1-A): track 0.00 -> 6.34 mm
- net Net-(D2-A): track 0.00 -> 6.33 mm
- net VBUS: track 10.9 -> 17.1 mm, vias 0 -> 2
- net /RP2040/VBUS_DETECT: track 0.00 -> 5.18 mm
- net /PreFIlterGND: track 3.88 -> 9.02 mm, vias 0 -> 3
- net /RP2040/~{RST}: track 0.00 -> 3.37 mm, vias 0 -> 2
- net /RP2040/SWCLK: track 0.00 -> 2.27 mm, vias 0 -> 2
- net /RP2040/SWDIO: track 0.00 -> 2.07 mm, vias 0 -> 2
- net /RP2040/RP2040/USB_D+: track 0.56 -> 2.42 mm, vias 1 -> 2
- net /RP2040/RP2040/USB_D-: track 0.61 -> 2.42 mm, vias 1 -> 2
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- added copper zone on In1.Cu, net /RP2040/3V3
Other:
- copper layers 2 -> 4

Commit message: Fix some errors, more routing
Parts:
- moved D6 19.2 mm to (123.0, 88.7), turned to 90 degrees
- moved R5 16.5 mm to (124.2, 88.8)
- moved FID1 2.90 mm to (144.9, 102.6)
Routing:
- net /Col0: track 1.22 -> 22.9 mm, vias 1 -> 3
- net /D1_OUT: track 0.00 -> 14.5 mm
- net +5V: track 19.0 -> 27.5 mm, vias 3 -> 4
- net GND: track 51.5 -> 44.0 mm, vias 40 -> 66
- net /RP2040/3V3: track 41.2 -> 44.6 mm, vias 12 -> 15
- net Net-(D6-A): track 0.00 -> 1.46 mm
- net /Row1: track 0.99 -> 2.06 mm, vias 1 -> 2
- net /Row0: track 1.14 -> 2.21 mm, vias 1 -> 2
- net /RP2040/~{RST}: track 3.37 -> 3.98 mm, vias 2 -> 3
- net /RP2040/RP2040/1V1: vias 1 -> 2
- net /PreFIlterGND: vias 3 -> 5
- net (no net): vias 0 -> 1
- added copper zone on In2.Cu, net /RP2040/RP2040/1V1

Commit message: Update todo's
Other:
- board text added: "TODO: Messure position for Key LED"
Changed lines of the file:
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@@
 		(layer "Edge.Cuts")
+	)
+	(gr_text "TODO: Messure position for Key LED"
+		(at 98.95 107.775 0)
+		(layer "F.Cu")
+		(effects
+			(font
+				(size 3 3)
+				(thickness 0.3)
+				(bold yes)
+			)
+			(justify left bottom)
+		)
 	)
 	(via

Commit message: Finish off routing
Parts:
- added FID2: Fiducial, Fiducial:Fiducial_1mm_Mask2mm, B.Cu at (134.1, 74.8)
- added TP1: Reset, TestPoint:TestPoint_Pad_D1.0mm, F.Cu at (156.2, 82.9)
- added TP2: Delay, TestPoint:TestPoint_Pad_D1.0mm, B.Cu at (155.2, 90.9)
- moved C2 2.87 mm to (132.9, 85.8), turned to -90 degrees
- moved D3 0.48 mm to (131.4, 89.5)
- moved D4 0.48 mm to (150.4, 89.5)
- moved C11 0.33 mm to (145.8, 83.1)
- moved R15 0.30 mm to (154.8, 88.6)
- moved R9 0.30 mm to (155.8, 88.6)
Routing:
- net /Row0: track 2.21 -> 43.7 mm, vias 2 -> 3
- net +5V: track 27.5 -> 60.8 mm, vias 4 -> 0
- net /TX0: track 1.08 -> 32.8 mm, vias 1 -> 3
- net /Row1: track 2.06 -> 32.0 mm
- net /Col0: track 22.9 -> 52.3 mm, vias 3 -> 4
- net /RP2040/RP2040/QSPI_~{CS}: track 7.64 -> 35.2 mm, vias 1 -> 3
- net /RP2040/RP2040/USB_D+: track 2.42 -> 26.2 mm
- net /RP2040/RP2040/USB_D-: track 2.42 -> 25.3 mm
- net /D2_OUT: track 0.00 -> 19.7 mm, vias 0 -> 2
- net /RP2040/RP2040/1V1: track 6.10 -> 25.3 mm, vias 2 -> 3
- net /RP2040/~{RST}: track 3.98 -> 20.3 mm
- net /RP2040/3V3: track 44.6 -> 57.6 mm, vias 15 -> 13
- net /RP2040/STATUS_LED_DO: track 1.04 -> 13.5 mm, vias 1 -> 2
- net /RP2040/SWDIO: track 2.07 -> 8.36 mm
- net /RP2040/SWCLK: track 2.27 -> 7.92 mm
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- added copper zone on In1.Cu, net /PreFIlterGND
- added copper zone on In2.Cu, net /PreFIlterGND
- added copper zone on In1.Cu, net /RP2040/RP2040/1V1
- added copper zone on In1.Cu, net GND
- added copper zone on In2.Cu, net GND
- removed copper zone on In2.Cu, net /RP2040/RP2040/1V1
Other:
- outline, holes or cut-outs redrawn
- board text added: "TODO: GET Missing 3D Model"
- board text removed: "TODO: Messure position for Key LED"

Commit message: Minor silk update
Parts:
- added TP3: OUT3, TestPoint:TestPoint_Pad_D1.0mm, B.Cu at (141.9, 95.8)
- added TP4: LED_DO, TestPoint:TestPoint_Pad_D1.0mm, F.Cu at (149.8, 73.7)
- TP1: value Reset -> RESET
- TP2: value Delay -> DELAY
Connections:
- net /D1_OUT renamed /Out1
- net /D2_OUT renamed /Out2
- D8 pad 2: /D3_OUT -> /Out3
Routing:
- net /Out3: track 0.00 -> 3.22 mm
- net /RP2040/LED_DO: track 0.00 -> 1.24 mm, vias 0 -> 1
Other:
- board text removed: "TODO: GET Missing 3D Model"

Commit message: Add board tabs
Parts:
- added T1: Tab, PCM_kikit:Tab, F.Cu at (140.9, 71.7)
- added T2: Tab, PCM_kikit:Tab, F.Cu at (121.9, 84.7)
- added T3: Tab, PCM_kikit:Tab, F.Cu at (159.9, 84.7)
- added T4: Tab, PCM_kikit:Tab, F.Cu at (140.9, 103.8)
